File: qwail56 v1/pcb/qwail56.kicad_sch (KiCad schematic)
At the start: 75 parts, among them J1 PJ-320A, SW1 CPG151101S11-16, SW10 CPG151101S11-16, SW11 CPG151101S11-16, SW12 CPG151101S11-16, SW13 CPG151101S11-16, SW14 CPG151101S11-16, SW15 CPG151101S11-16, SW16 CPG151101S11-16, SW17 CPG151101S11-16, SW18 CPG151101S11-16, SW19 CPG151101S11-16, SW2 CPG151101S11-16, SW20 CPG151101S11-16, SW21 CPG151101S11-16, SW22 CPG151101S11-16, SW23 CPG151101S11-16, SW24 CPG151101S11-16, SW25 CPG151101S11-16, SW26 CPG151101S11-16, SW27 CPG151101S11-16, SW28 CPG151101S11-16, SW29 EVQWGD001, SW3 CPG151101S11-16, SW30 EVQWGD001, SW31 EC11E, SW4 CPG151101S11-16, SW5 CPG151101S11-16, SW6 CPG151101S11-16, SW7 CPG151101S11-16, SW8 CPG151101S11-16, SW9 CPG151101S11-16, U1 Pico

Commit message: Add files via upload
Parts:
- SW31: footprint qwail56:EC11E_reversible -> qwail56:Rotary_Encoder_EC11E_reversible
Changed lines of the file:
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@@
       (effects (font (size 1.27 1.27)))
     )
-    (property "Footprint" "qwail56:EC11E_reversible" (at 53.34 192.786 0)
+    (property "Footprint" "qwail56:Rotary_Encoder_EC11E_reversible" (at 53.34 192.786 0)
       (effects (font (size 1.27 1.27)) hide)
     )
